Commit message: Add files via upload

File: motoman_sda20d_support/urdf/motoman_sda20d.urdf (robot description, URDF)
Before this commit: robot motoman_sda20d, 16 links, 15 joints
Joints:
- joint arm_left_joint_1_s: axis 0 0 1 -> 0 0 -1; limit lower=-2.9670 upper=2.9670 effort=0 velocity=2.4434 -> lower=-3.1400246620178223 upper=3.1400246620178223 effort=0 velocity=0.9076052904129028
- joint arm_left_joint_2_l: axis 0 0 1 -> 0 0 -1; limit lower=-2.9670 upper=2.9670 effort=0 velocity=2.4434 -> lower=-1.9198451042175293 upper=1.9198451042175293 effort=0 velocity=0.7968177795410156
- joint arm_left_joint_3_e: limit lower=-2.9670 upper=2.9670 effort=0 velocity=2.4434 -> lower=-2.966156244277954 upper=2.966156244277954 effort=0 velocity=1.0396981239318848
- joint arm_left_joint_4_u: axis 0 0 1 -> 0 0 -1; limit lower=-2.9670 upper=2.9670 effort=0 velocity=2.4434 -> lower=-2.268928050994873 upper=2.268928050994873 effort=0 velocity=1.1888351440429688
- joint arm_left_joint_5_r: axis 0 0 -1 -> 0 0 1; limit lower=-2.9670 upper=2.9670 effort=0 velocity=2.4434 -> lower=-3.140711545944214 upper=3.140711545944214 effort=0 velocity=1.5719505548477173
- joint arm_left_joint_6_b: axis 0 1 0 -> 0 -1 0; limit lower=-2.9670 upper=2.9670 effort=0 velocity=2.4434 -> lower=-1.9177645444869995 upper=1.9177645444869995 effort=0 velocity=1.7428147792816162
- joint arm_left_joint_7_t: axis 0 0 -1 -> 0 0 1; limit lower=-2.9670 upper=2.9670 effort=0 velocity=2.4434 -> lower=-3.1383140087127686 upper=3.1383140087127686 effort=0 velocity=2.0453076362609863
- joint arm_right_joint_1_s: limit lower=-2.9670 upper=2.9670 effort=0 velocity=2.4434 -> lower=-3.1400246620178223 upper=3.1400246620178223 effort=0 velocity=0.9076052904129028
- joint arm_right_joint_2_l: limit lower=-2.9670 upper=2.9670 effort=0 velocity=2.4434 -> lower=-1.9191462993621826 upper=1.9191462993621826 effort=0 velocity=0.7968177795410156
- joint arm_right_joint_3_e: limit lower=-2.9670 upper=2.9670 effort=0 velocity=2.4434 -> lower=-2.9661734104156494 upper=2.9661734104156494 effort=0 velocity=1.0396981239318848
- joint arm_right_joint_4_u: limit lower=-2.9670 upper=2.9670 effort=0 velocity=2.4434 -> lower=-2.2681779861450195 upper=2.2681779861450195 effort=0 velocity=1.1888351440429688
- joint arm_right_joint_5_r: limit lower=-2.9670 upper=2.9670 effort=0 velocity=2.4434 -> lower=-3.140711545944214 upper=3.140711545944214 effort=0 velocity=1.5719505548477173
- joint arm_right_joint_6_b: limit lower=-2.9670 upper=2.9670 effort=0 velocity=2.4434 -> lower=-1.9177796840667725 upper=1.9177796840667725 effort=0 velocity=1.7428147792816162
- joint arm_right_joint_7_t: limit lower=-2.9670 upper=2.9670 effort=0 velocity=2.4434 -> lower=-3.1383140087127686 upper=3.1383140087127686 effort=0 velocity=2.0453076362609863
- joint torso_joint_b1: limit lower=-2.9670 upper=2.9670 effort=0 velocity=2.4434 -> lower=-1.5555423498153687 upper=1.5555423498153687 effort=0 velocity=2.4434

Commit message: Add files via upload

File: motoman_sda20d_support/urdf/motoman_sda20d.urdf (robot description, URDF)
Before this commit: robot motoman_sda20d, 16 links, 15 joints
Links:
- removed link arm_left_link_1_s
- removed link arm_left_link_2_l
- removed link arm_left_link_3_e
- removed link arm_left_link_4_u
- removed link arm_left_link_5_r
- removed link arm_left_link_6_b
- removed link arm_left_link_7_t
- removed link arm_right_link_1_s
- removed link arm_right_link_2_l
- removed link arm_right_link_3_e
- removed link arm_right_link_4_u
- removed link arm_right_link_5_r
- removed link arm_right_link_6_b
- removed link arm_right_link_7_t
- added link arm_left_link_b; collision mesh filename=package://motoman_sda20d_support/meshes/arm_link_b.STL; visual mesh filename=package://motoman_sda20d_support/meshes/arm_link_b.STL
- added link arm_left_link_e; collision mesh filename=package://motoman_sda20d_support/meshes/arm_link_e.STL; visual mesh filename=package://motoman_sda20d_support/meshes/arm_link_e.STL
- added link arm_left_link_l; collision mesh filename=package://motoman_sda20d_support/meshes/arm_link_l.STL; visual mesh filename=package://motoman_sda20d_support/meshes/arm_link_l.STL
- added link arm_left_link_r; collision mesh filename=package://motoman_sda20d_support/meshes/arm_link_r.STL; visual mesh filename=package://motoman_sda20d_support/meshes/arm_link_r.STL
- added link arm_left_link_s; collision mesh filename=package://motoman_sda20d_support/meshes/arm_link_s.STL; visual mesh filename=package://motoman_sda20d_support/meshes/arm_link_s.STL
- added link arm_left_link_t; collision mesh filename=package://motoman_sda20d_support/meshes/arm_link_t.STL; visual mesh filename=package://motoman_sda20d_support/meshes/arm_link_t.STL
- added link arm_left_link_u; collision mesh filename=package://motoman_sda20d_support/meshes/arm_link_u.STL; visual mesh filename=package://motoman_sda20d_support/meshes/arm_link_u.STL
- added link arm_right_link_b; collision mesh filename=package://motoman_sda20d_support/meshes/arm_link_b.STL; visual mesh filename=package://motoman_sda20d_support/meshes/arm_link_b.STL
- added link arm_right_link_e; collision mesh filename=package://motoman_sda20d_support/meshes/arm_link_e.STL; visual mesh filename=package://motoman_sda20d_support/meshes/arm_link_e.STL
- added link arm_right_link_l; collision mesh filename=package://motoman_sda20d_support/meshes/arm_link_l.STL; visual mesh filename=package://motoman_sda20d_support/meshes/arm_link_l.STL
- added link arm_right_link_r; collision mesh filename=package://motoman_sda20d_support/meshes/arm_link_r.STL; visual mesh filename=package://motoman_sda20d_support/meshes/arm_link_r.STL
- added link arm_right_link_s; collision mesh filename=package://motoman_sda20d_support/meshes/arm_link_s.STL; visual mesh filename=package://motoman_sda20d_support/meshes/arm_link_s.STL
- added link arm_right_link_t; collision mesh filename=package://motoman_sda20d_support/meshes/arm_link_t.STL; visual mesh filename=package://motoman_sda20d_support/meshes/arm_link_t.STL
- added link arm_right_link_u; collision mesh filename=package://motoman_sda20d_support/meshes/arm_link_u.STL; visual mesh filename=package://motoman_sda20d_support/meshes/arm_link_u.STL
- link base_link: mass 29.711 -> None
- link torso_link_b1: mass 36.439 -> None
Joints:
- removed joint arm_left_joint_1_s
- removed joint arm_left_joint_2_l
- removed joint arm_left_joint_3_e
- removed joint arm_left_joint_4_u
- removed joint arm_left_joint_5_r
- removed joint arm_left_joint_6_b
- removed joint arm_left_joint_7_t
- removed joint arm_right_joint_1_s
- removed joint arm_right_joint_2_l
- removed joint arm_right_joint_3_e
- removed joint arm_right_joint_4_u
- removed joint arm_right_joint_5_r
- removed joint arm_right_joint_6_b
- removed joint arm_right_joint_7_t
- added joint arm_left_joint_b: type revolute, parent arm_left_link_r, child arm_left_link_b, origin xyz=0 0 -0.181 rpy=3.14159265359 1.57079632679 0, axis 0 -1 0, limit lower=-1.917 upper=1.917 effort=1000 velocity=1.74
- added joint arm_left_joint_e: type revolute, parent arm_left_link_l, child arm_left_link_e, origin xyz=0.2659 0 0.04877 rpy=-1.57079632679 3.14159265359 1.57079632679, axis 0 0 -1, limit lower=-2.966 upper=2.966 effort=1000 velocity=1.039
- added joint arm_left_joint_l: type revolute, parent arm_left_link_s, child arm_left_link_l, origin xyz=0 -0.0571 -0.3145 rpy=-1.57079632679 1.57079632679 0, axis 0 0 -1, limit lower=-1.92 upper=1.92 effort=1000 velocity=0.796
- added joint arm_left_joint_r: type revolute, parent arm_left_link_u, child arm_left_link_r, origin xyz=0.26425 0 0.0015 rpy=-1.57079632679 0 1.57079632679, axis 0 0 1, limit lower=-3.14 upper=3.14 effort=1000 velocity=1.5719
- added joint arm_left_joint_s: type revolute, parent torso_link_b1, child arm_left_link_s, origin xyz=0.15 0.075 0.2984 rpy=1.57079632679 -0.0 0, axis 0 0 -1, limit lower=-3.14 upper=3.14 effort=1000 velocity=0.9086
- added joint arm_left_joint_t: type revolute, parent arm_left_link_b, child arm_left_link_t, origin xyz=0.16725 0.02775 0 rpy=3.14159265359 1.57079632679 0, axis 0 0 1, limit lower=-3.1383 upper=3.1383 effort=1000 velocity=2.0453
- added joint arm_left_joint_u: type revolute, parent arm_left_link_e, child arm_left_link_u, origin xyz=0 0.0494 -0.2441 rpy=1.57079632679 1.57079632679 0, axis 0 0 -1, limit lower=-2.2689 upper=2.2689 effort=1000 velocity=1.188
- added joint arm_right_joint_b: type revolute, parent arm_right_link_r, child arm_right_link_b, origin xyz=0 0 -0.181 rpy=3.14159265359 1.57079632679 0, axis 0 1 0, limit lower=-1.917 upper=1.917 effort=1000 velocity=1.74
- added joint arm_right_joint_e: type revolute, parent arm_right_link_l, child arm_right_link_e, origin xyz=0.2659 0 0.04877 rpy=-1.57079632679 3.14159265359 1.57079632679, axis 0 0 1, limit lower=-2.966 upper=2.966 effort=1000 velocity=1.039
- added joint arm_right_joint_l: type revolute, parent arm_right_link_s, child arm_right_link_l, origin xyz=0 -0.0571 -0.3145 rpy=-1.57079632679 1.57079632679 0, axis 0 0 1, limit lower=-1.92 upper=1.92 effort=1000 velocity=0.796
- added joint arm_right_joint_r: type revolute, parent arm_right_link_u, child arm_right_link_r, origin xyz=0.26425 0 0.0015 rpy=-1.57079632679 0 1.57079632679, axis 0 0 -1, limit lower=-3.14 upper=3.14 effort=1000 velocity=1.5719
- added joint arm_right_joint_s: type revolute, parent torso_link_b1, child arm_right_link_s, origin xyz=0.15 -0.075 0.2984 rpy=-1.57079632679 3.14159265359 0, axis 0 0 1, limit lower=-3.14 upper=3.14 effort=1000 velocity=0.9086
- added joint arm_right_joint_t: type revolute, parent arm_right_link_b, child arm_right_link_t, origin xyz=0.16725 0.02775 0 rpy=3.14159265359 1.57079632679 0, axis 0 0 -1, limit lower=-3.1383 upper=3.1383 effort=1000 velocity=2.0453
- added joint arm_right_joint_u: type revolute, parent arm_right_link_e, child arm_right_link_u, origin xyz=0 0.0494 -0.2441 rpy=1.57079632679 1.57079632679 0, axis 0 0 1, limit lower=-2.2689 upper=2.2689 effort=1000 velocity=1.188
- joint torso_joint_b1: limit lower=-1.5555423498153687 upper=1.5555423498153687 effort=0 velocity=2.4434 -> lower=-1.5555423498153687 upper=1.5555423498153687 effort=1000 velocity=2.4434
