Commit message: Add files via upload

File: motoman_sda20d_support/urdf/motoman_sda20d.urdf (robot description, URDF)
Before this commit: robot motoman_sda20d, 16 links, 15 joints
Links:
- removed link arm_left_link_b
- removed link arm_left_link_e
- removed link arm_left_link_l
- removed link arm_left_link_r
- removed link arm_left_link_s
- removed link arm_left_link_t
- removed link arm_left_link_u
- removed link arm_right_link_b
- removed link arm_right_link_e
- removed link arm_right_link_l
- removed link arm_right_link_r
- removed link arm_right_link_s
- removed link arm_right_link_t
- removed link arm_right_link_u
- added link arm_left_link_1_s, mass 12.738; collision mesh filename=package://motoman_sda20d_support/meshes/arm_left_link_1_s.S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; visual mesh filename=package://motoman_sda20d_support/meshes/arm_left_link_1_s.S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
- added link arm_left_link_2_l, mass 6.6303; collision mesh filename=package://motoman_sda20d_support/meshes/arm_left_link_2_l.S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; visual mesh filename=package://motoman_sda20d_support/meshes/arm_left_link_2_l.S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
- added link arm_left_link_3_e, mass 7.0076; collision mesh filename=package://motoman_sda20d_support/meshes/arm_left_link_3_e.S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; visual mesh filename=package://motoman_sda20d_support/meshes/arm_left_link_3_e.S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
- added link arm_left_link_4_u, mass 4.4681; collision mesh filename=package://motoman_sda20d_support/meshes/arm_left_link_4_u.S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; visual mesh filename=package://motoman_sda20d_support/meshes/arm_left_link_4_u.S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
- added link arm_left_link_5_r, mass 2.5196; collision mesh filename=package://motoman_sda20d_support/meshes/arm_left_link_5_r.S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; visual mesh filename=package://motoman_sda20d_support/meshes/arm_left_link_5_r.S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
- added link arm_left_link_6_b, mass 2.1679; collision mesh filename=package://motoman_sda20d_support/meshes/arm_left_link_6_b.S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; visual mesh filename=package://motoman_sda20d_support/meshes/arm_left_link_6_b.S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
- added link arm_left_link_7_t, mass 0.107191529942716; collision mesh filename=package://motoman_sda20d_support/meshes/arm_left_link_7_t.S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; visual mesh filename=package://motoman_sda20d_support/meshes/arm_left_link_7_t.S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
- added link arm_right_link_1_s, mass 12.7382287673505; collision mesh filename=package://motoman_sda20d_support/meshes/arm_right_link_1_s.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; visual mesh filename=package://motoman_sda20d_support/meshes/arm_right_link_1_s.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
- added link arm_right_link_2_l, mass 6.6303; collision mesh filename=package://motoman_sda20d_support/meshes/arm_right_link_2_l.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; visual mesh filename=package://motoman_sda20d_support/meshes/arm_right_link_2_l.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
- added link arm_right_link_3_e, mass 7.0076; collision mesh filename=package://motoman_sda20d_support/meshes/arm_right_link_3_e.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; visual mesh filename=package://motoman_sda20d_support/meshes/arm_right_link_3_e.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
- added link arm_right_link_4_u, mass 4.4681; collision mesh filename=package://motoman_sda20d_support/meshes/arm_right_link_4_u.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; visual mesh filename=package://motoman_sda20d_support/meshes/arm_right_link_4_u.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
- added link arm_right_link_5_r, mass 2.51962025325968; collision mesh filename=package://motoman_sda20d_support/meshes/arm_right_link_5_r.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; visual mesh filename=package://motoman_sda20d_support/meshes/arm_right_link_5_r.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
- added link arm_right_link_6_b, mass 2.1679; collision mesh filename=package://motoman_sda20d_support/meshes/arm_right_link_6_b.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; visual mesh filename=package://motoman_sda20d_support/meshes/arm_right_link_6_b.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
- added link arm_right_link_7_t, mass 0.10719; collision mesh filename=package://motoman_sda20d_support/meshes/arm_right_link_7_t.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; visual mesh filename=package://motoman_sda20d_support/meshes/arm_right_link_7_t.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
- link base_link: mass None -> 29.711
- link torso_link_b1: mass None -> 36.439
Joints:
- removed joint arm_left_joint_b
- removed joint arm_left_joint_e
- removed joint arm_left_joint_l
- removed joint arm_left_joint_r
- removed joint arm_left_joint_s
- removed joint arm_left_joint_t
- removed joint arm_left_joint_u
- removed joint arm_right_joint_b
- removed joint arm_right_joint_e
- removed joint arm_right_joint_l
- removed joint arm_right_joint_r
- removed joint arm_right_joint_s
- removed joint arm_right_joint_t
- removed joint arm_right_joint_u
- added joint arm_left_joint_1_s: type revolute, parent torso_link_b1, child arm_left_link_1_s, origin xyz=0.149999999999999 0.075 0.2984 rpy=1.5707963267949 0 0, axis 0 0 -1, limit lower=-3.1400246620178223 upper=3.1400246620178223 effort=0 velocity=0.9076052904129028
- added joint arm_left_joint_2_l: type revolute, parent arm_left_link_1_s, child arm_left_link_2_l, origin xyz=0 -0.0571 -0.3145 rpy=-1.5707963267949 1.5707963267949 0, axis 0 0 -1, limit lower=-1.9198451042175293 upper=1.9198451042175293 effort=0 velocity=0.7968177795410156
- added joint arm_left_joint_3_e: type revolute, parent arm_left_link_2_l, child arm_left_link_3_e, origin xyz=0.2659 0 0.0487700000000001 rpy=-1.5707963267949 3.141592654 1.5707963267949, axis 0 0 -1, limit lower=-2.966156244277954 upper=2.966156244277954 effort=0 velocity=1.0396981239318848
- added joint arm_left_joint_4_u: type revolute, parent arm_left_link_3_e, child arm_left_link_4_u, origin xyz=0 0.0494000000000001 -0.2441 rpy=1.5707963267949 1.5707963267949 0, axis 0 0 -1, limit lower=-2.268928050994873 upper=2.268928050994873 effort=0 velocity=1.1888351440429688
- added joint arm_left_joint_5_r: type revolute, parent arm_left_link_4_u, child arm_left_link_5_r, origin xyz=0.26425 0 0.00150000000000017 rpy=-1.5707963267949 0 1.5707963267949, axis 0 0 1, limit lower=-3.140711545944214 upper=3.140711545944214 effort=0 velocity=1.5719505548477173
- added joint arm_left_joint_6_b: type revolute, parent arm_left_link_5_r, child arm_left_link_6_b, origin xyz=0 0 -0.181 rpy=3.14159265358979 1.5707963267949 0, axis 0 -1 0, limit lower=-1.9177645444869995 upper=1.9177645444869995 effort=0 velocity=1.7428147792816162
- added joint arm_left_joint_7_t: type revolute, parent arm_left_link_6_b, child arm_left_link_7_t, origin xyz=0.16725 0.0277499999999999 0 rpy=3.14159265358979 1.5707963267949 0, axis 0 0 1, limit lower=-3.1383140087127686 upper=3.1383140087127686 effort=0 velocity=2.0453076362609863
- added joint arm_right_joint_1_s: type revolute, parent torso_link_b1, child arm_right_link_1_s, origin xyz=0.15 -0.075 0.2984 rpy=-1.5707963267949 3.141592654 0, axis 0 0 1, limit lower=-3.1400246620178223 upper=3.1400246620178223 effort=0 velocity=0.9076052904129028
- added joint arm_right_joint_2_l: type revolute, parent arm_right_link_1_s, child arm_right_link_2_l, origin xyz=0 -0.0571 -0.3145 rpy=-1.5707963267949 1.5707963267949 0, axis 0 0 1, limit lower=-1.9191462993621826 upper=1.9191462993621826 effort=0 velocity=0.7968177795410156
- added joint arm_right_joint_3_e: type revolute, parent arm_right_link_2_l, child arm_right_link_3_e, origin xyz=0.2659 0 0.04877 rpy=1.5707963267949 0 -1.5707963267949, axis 0 0 1, limit lower=-2.9661734104156494 upper=2.9661734104156494 effort=0 velocity=1.0396981239318848
- added joint arm_right_joint_4_u: type revolute, parent arm_right_link_3_e, child arm_right_link_4_u, origin xyz=0 0.0494 -0.2441 rpy=1.5707963267949 1.5707963267949 0, axis 0 0 1, limit lower=-2.2681779861450195 upper=2.2681779861450195 effort=0 velocity=1.1888351440429688
- added joint arm_right_joint_5_r: type revolute, parent arm_right_link_4_u, child arm_right_link_5_r, origin xyz=0.26425 0 0.0015 rpy=-1.5707963267949 0 1.5707963267949, axis 0 0 -1, limit lower=-3.140711545944214 upper=3.140711545944214 effort=0 velocity=1.5719505548477173
- added joint arm_right_joint_6_b: type revolute, parent arm_right_link_5_r, child arm_right_link_6_b, origin xyz=0 -0.0317499999999999 -0.181 rpy=1.5707963267949 1.5707963267949 0, axis 0 0 1, limit lower=-1.9177796840667725 upper=1.9177796840667725 effort=0 velocity=1.7428147792816162
- added joint arm_right_joint_7_t: type revolute, parent arm_right_link_6_b, child arm_right_link_7_t, origin xyz=0.16725 0 -0.004 rpy=-1.5707963267949 0 1.5707963267949, axis 0 0 -1, limit lower=-3.1383140087127686 upper=3.1383140087127686 effort=0 velocity=2.0453076362609863
- joint torso_joint_b1: limit lower=-1.5555423498153687 upper=1.5555423498153687 effort=1000 velocity=2.4434 -> lower=-1.5555423498153687 upper=1.5555423498153687 effort=0 velocity=2.4434

File: motoman_sda20d_support/urdf/motoman_sda20d.xacro (robot description, xacro)
@@ -1,87 +1,853 @@
 <?xml version="1.0"?>
 <robot xmlns:xacro="http://www.ros.org/wiki/xacro" name="motoman_sda20d">
-  <link name="base_link">
-    <visual>
-      <origin xyz="0 0 0" rpy="0 0 0" />
-      <geometry>
-        <mesh filename="package://motoman_sda20d_support/meshes/base_link.STL" />
-      </geometry>
-      <material name="">
-        <color rgba="0.79216 0.81 0.93 1" />
-      </material>
-    </visual>
-    <collision>
-      <origin xyz="0 0 0" rpy="0 0 0" />
-      <geometry>
-        <mesh filename="package://motoman_sda20d_support/meshes/base_link.STL" />
-      </geometry>
-    </collision>
-  </link>
-  <link name="torso_link_b1">
-    <visual>
-      <origin xyz="0 0 0" rpy="0 0 0" />
-      <geometry>
-        <mesh filename="package://motoman_sda20d_support/meshes/torso_link_b1.STL" />
-      </geometry>
-      <material name="">
-        <color rgba="0.79 0.81 1 1" />
-      </material>
-    </visual>
-    <collision>
-      <origin xyz="0 0 0" rpy="0 0 0" />
-      <geometry>
-        <mesh filename="package://motoman_sda20d_support/meshes/torso_link_b1.STL" />
-      </geometry>
-    </collision>
-  </link>
-  <joint name="torso_joint_b1" type="revolute">
-    <origin xyz="0 0 0.2765" rpy="0 0 0" />
-    <parent link="base_link" />
-    <child link="torso_link_b1" />
-    <axis xyz="0 0 1" />
-    <limit effort="1000" lower="-1.5555423498153687" upper="1.5555423498153687" velocity="2.4434"/>
-  </joint>
-  <xacro:macro name="motoman_arm_link" params="side link_name rgba parent xyz rpy axis lower upper velocity reflect" >
-  <link name="arm_${side}_link_${link_name}">
-    <visual>
-      <origin xyz="0 0 0" rpy="0 0 0" />
-      <geometry>
-        <mesh filename="package://motoman_sda20d_support/meshes/arm_link_${link_name}.STL" />
-      </geometry>
-      <material name="">
-        <color rgba="${rgba}" />
-      </material>
-    </visual>
-    <collision>
-      <origin xyz="0 0 0" rpy="0 0 0" />
-      <geometry>
-        <mesh filename="package://motoman_sda20d_support/meshes/arm_link_${link_name}.STL" />
-      </geometry>
-    </collision>
-  </link>
-  <joint name="arm_${side}_joint_${link_name}" type="revolute">
-    <origin xyz="${xyz}" rpy="${rpy}" />
-    <parent link="${parent}" />
-    <child link="arm_${side}_link_${link_name}" />
-    <axis xyz="${axis}" />
-    <limit effort="1000" lower="${lower}" upper="${upper}" velocity="${velocity}"/>
-  </joint>
-  </xacro:macro>
-  <xacro:macro name="motoman_arm_side" params="side">
-  <xacro:if value="${side=='left'}">
-  <xacro:property name="reflect" value="1"/>
-  </xacro:if>
-  <xacro:unless value="${side=='left'}">
-  <xacro:property name="reflect" value="-1"/>
-  </xacro:unless>
-  <xacro:motoman_arm_link side="${side}" link_name="s" rgba="0.79 0.81 0.93 1" parent="torso_link_b1" xyz="0.15 ${0.075 * reflect} 0.2984" rpy="${pi/2* reflect} ${(pi/2 * (reflect - 1)) * -1} 0" axis="0 0 ${reflect * -1}" lower="-3.14" upper="3.14" velocity="0.9086" reflect="${reflect}"/>
-  <xacro:motoman_arm_link side="${side}" link_name="l" rgba="0.79 0.81 1 1" parent="arm_${side}_link_s" xyz="0 -0.0571 -0.3145" rpy="-${pi/2} ${pi/2} 0" axis="0 0 ${reflect * -1}" lower="-1.92" upper="1.92" velocity="0.796" reflect="${reflect}"/>
-  <xacro:motoman_arm_link side="${side}" link_name="e" rgba="0.79 0.81 0.93 1" parent="arm_${side}_link_l" xyz="0.2659 0 0.04877" rpy="-${pi/2} ${pi} ${pi/2}" axis="0 0 ${reflect * -1}" lower="-2.966" upper="2.966" velocity="1.039" reflect="${reflect}"/>
-  <xacro:motoman_arm_link side="${side}" link_name="u" rgba="0.79 0.81 1 1" parent="arm_${side}_link_e" xyz="0 0.0494 -0.2441" rpy="${pi/2} ${pi/2} 0" axis="0 0 ${reflect * -1}" lower="-2.2689" upper="2.2689" velocity="1.188" reflect="${reflect}"/>
-  <xacro:motoman_arm_link side="${side}" link_name="r" rgba="0.79 0.81 0.93 1" parent="arm_${side}_link_u" xyz="0.26425 0 0.0015" rpy="-${pi/2} 0 ${pi/2}" axis="0 0 ${reflect * 1}" lower="-3.14" upper="3.14" velocity="1.5719" reflect="${reflect}"/>
-  <xacro:motoman_arm_link side="${side}" link_name="b" rgba="0.79 0.81 1 1" parent="arm_${side}_link_r" xyz="0 0 -0.181" rpy="${pi} ${pi/2} 0" axis="0 ${reflect * -1} 0" lower="-1.917" upper="1.917" velocity="1.74" reflect="${reflect}"/>
-  <xacro:motoman_arm_link side="${side}" link_name="t" rgba="0.79 0.81 0.93 1" parent="arm_${side}_link_b" xyz="0.16725 0.02775 0" rpy="${pi} ${pi/2} 0" axis="0 0 ${reflect * 1}" lower="-3.1383" upper="3.1383" velocity="2.0453" reflect="${reflect}"/>
-  </xacro:macro>
-  <xacro:motoman_arm_side side="left"/>
-  <xacro:motoman_arm_side side="right"/>
+  <link
+    name="base_link">
+    <inertial>
+      <origin
+        xyz="-0.10775 -4.7555E-05 0.10955"
+        rpy="0 0 0" />
+      <mass
+        value="29.711" />
+      <inertia
+        ixx="0.37202"
+        ixy="-0.00060974"
+        ixz="-0.024001"
+        iyy="0.77862"
+        iyz="4.9206E-05"
+        izz="0.84078" />
+    </inertial>
+    <visual>
+      <origin
+        xyz="0 0 0"
+        rpy="0 0 0" />
+      <geometry>
+        <mesh
+          filename="package://motoman_sda20d_support/meshes/base_link.STL" />
+      </geometry>
+      <material
+        name="">
+        <color
+          rgba="0.79216 0.81961 0.93333 1" />
+      </material>
+    </visual>
+    <collision>
+      <origin
+        xyz="0 0 0"
+        rpy="0 0 0" />
+      <geometry>
+        <mesh
+          filename="package://motoman_sda20d_support/meshes/base_link.STL" />
+      </geometry>
+    </collision>
+  </link>
+  <link
+    name="torso_link_b1">
+    <inertial>
+      <origin
+        xyz="0.026706 1.1222E-05 0.19713"
+        rpy="0 0 0" />
+      <mass
+        value="36.439" />
+      <inertia
+        ixx="0.62924"
+        ixy="7.5604E-05"
+        ixz="-0.065715"
+        iyy="0.97273"
+        iyz="7.3187E-05"
+        izz="0.67513" />
+    </inertial>
+    <visual>
+      <origin
+        xyz="0 0 0"
+        rpy="0 0 0" />
+      <geometry>
+        <mesh
+          filename="package://motoman_sda20d_support/meshes/torso_link_b1.STL" />
+      </geometry>
+      <material
+        name="">
+        <color
+          rgba="0.79216 0.81961 1 1" />
+      </material>
+    </visual>
+    <collision>
+      <origin
+        xyz="0 0 0"
+        rpy="0 0 0" />
+      <geometry>
+        <mesh
+          filename="package://motoman_sda20d_support/meshes/torso_link_b1.STL" />
+      </geometry>
+    </collision>
+  </link>
+  <joint
+    name="torso_joint_b1"
+    type="revolute">
+    <origin
+      xyz="0 0 0.2765"
+      rpy="0 0 0" />
+    <parent
+      link="base_link" />
+    <child
+      link="torso_link_b1" />
+    <axis
+      xyz="0 0 1" />
+    <limit effort="0" lower="-1.5555423498153687" upper="1.5555423498153687" velocity="2.4434"/>
+  </joint>
+  <link
+    name="arm_left_link_1_s">
+    <inertial>
+      <origin
+        xyz="-4.4465E-06 0.014517 -0.19101"
+        rpy="0 0 0" />
+      <mass
+        value="12.738" />
+      <inertia
+        ixx="0.22105"
+        ixy="1.8397E-06"
+        ixz="-7.8564E-06"
+        iyy="0.22442"
+        iyz="0.016414"
+        izz="0.069643" />
+    </inertial>
+    <visual>
+      <origin
+        xyz="0 0 0"
+        rpy="0 0 0" />
+      <geometry>
+        <mesh
+          filename="package://motoman_sda20d_support/meshes/arm_left_link_1_s.STL" />
+      </geometry>
+      <material
+        name="">
+        <color
+          rgba="0.79216 0.81961 0.93333 1" />
+      </material>
+    </visual>
+    <collision>
+      <origin
+        xyz="0 0 0"
+        rpy="0 0 0" />
+      <geometry>
+        <mesh
+          filename="package://motoman_sda20d_support/meshes/arm_left_link_1_s.STL" />
+      </geometry>
+    </collision>
+  </link>
+  <joint
+    name="arm_left_joint_1_s"
+    type="revolute">
+    <origin
+      xyz="0.149999999999999 0.075 0.2984"
+      rpy="1.5707963267949 0 0" />
+    <parent
+      link="torso_link_b1" />
+    <child
+      link="arm_left_link_1_s" />
+    <axis
+      xyz="0 0 -1" />
+    <limit effort="0" lower="-3.1400246620178223" upper="3.1400246620178223" velocity="0.9076052904129028"/>
+  </joint>
+  <link
+    name="arm_left_link_2_l">
+    <inertial>
+      <origin
+        xyz="0.099179 2.1877E-05 0.0070227"
+        rpy="0 0 0" />
+      <mass
+        value="6.6303" />
+      <inertia
+        ixx="0.034667"
+        ixy="-7.854E-06"
+        ixz="-0.0228"
+        iyy="0.089109"
+        iyz="-5.3344E-06"
+        izz="0.091218" />
+    </inertial>
+    <visual>
+      <origin
+        xyz="0 0 0"
+        rpy="0 0 0" />
+      <geometry>
+        <mesh
+          filename="package://motoman_sda20d_support/meshes/arm_left_link_2_l.STL" />
+      </geometry>
+      <material
+        name="">
+        <color
+          rgba="0.79216 0.81961 1 1" />
+      </material>
+    </visual>
+    <collision>
+      <origin
+        xyz="0 0 0"
+        rpy="0 0 0" />
+      <geometry>
+        <mesh
+          filename="package://motoman_sda20d_support/meshes/arm_left_link_2_l.STL" />
+      </geometry>
+    </collision>
+  </link>
+  <joint
+    name="arm_left_joint_2_l"
+    type="revolute">
+    <origin
+      xyz="0 -0.0571 -0.3145"
+      rpy="-1.5707963267949 1.5707963267949 0" />
+    <parent
+      link="arm_left_link_1_s" />
+    <child
+      link="arm_left_link_2_l" />
+    <axis
+      xyz="0 0 -1" />
+    <limit effort="0" lower="-1.9198451042175293" upper="1.9198451042175293" velocity="0.7968177795410156"/>
+  </joint>
+  <link
+    name="arm_left_link_3_e">
+    <inertial>
+      <origin
+        xyz="-2.2325E-06 -0.017232 -0.15134"
+        rpy="0 0 0" />
+      <mass
+        value="7.0076" />
+      <inertia
+        ixx="0.077721"
+        ixy="-1.9693E-08"
+        ixz="3.9327E-07"
+        iyy="0.075759"
+        iyz="-0.0060104"
+        izz="0.027096" />
+    </inertial>
+    <visual>
+      <origin
+        xyz="0 0 0"
+        rpy="0 0 0" />
+      <geometry>
+        <mesh
+          filename="package://motoman_sda20d_support/meshes/arm_left_link_3_e.STL" />
+      </geometry>
+      <material
+        name="">
+        <color
+          rgba="0.79216 0.81961 0.93333 1" />
+      </material>
+    </visual>
+    <collision>
+      <origin
+        xyz="0 0 0"
+        rpy="0 0 0" />
+      <geometry>
+        <mesh
+          filename="package://motoman_sda20d_support/meshes/arm_left_link_3_e.STL" />
+      </geometry>
+    </collision>
+  </link>
+  <joint
+    name="arm_left_joint_3_e"
+    type="revolute">
+    <origin
+      xyz="0.2659 0 0.0487700000000001"
+      rpy="-1.5707963267949 3.141592654 1.5707963267949" />
+    <parent
+      link="arm_left_link_2_l" />
+    <child
+      link="arm_left_link_3_e" />
+    <axis
+      xyz="0 0 -1" />
+    <limit effort="0" lower="-2.966156244277954" upper="2.966156244277954" velocity="1.0396981239318848"/>
+  </joint>
+  <link
+    name="arm_left_link_4_u">
+    <inertial>
+      <origin
+        xyz="0.084741 -1.2964E-05 -0.031047"
+        rpy="0 0 0" />
+      <mass
+        value="4.4681" />
+      <inertia
+        ixx="0.0122"
+        ixy="1.1308E-05"
+        ixz="-0.006865"
+        iyy="0.048201"
+        iyz="3.1167E-06"
+        izz="0.049778" />
+    </inertial>
+    <visual>
+      <origin
+        xyz="0 0 0"
+        rpy="0 0 0" />
+      <geometry>
+        <mesh
+          filename="package://motoman_sda20d_support/meshes/arm_left_link_4_u.STL" />
+      </geometry>
+      <material
+        name="">
+        <color
+          rgba="0.79216 0.81961 1 1" />
+      </material>
+    </visual>
+    <collision>
+      <origin
+        xyz="0 0 0"
+        rpy="0 0 0" />
+      <geometry>
+        <mesh
+          filename="package://motoman_sda20d_support/meshes/arm_left_link_4_u.STL" />
+      </geometry>
+    </collision>
+  </link>
+  <joint
+    name="arm_left_joint_4_u"
+    type="revolute">
+    <origin
+      xyz="0 0.0494000000000001 -0.2441"
+      rpy="1.5707963267949 1.5707963267949 0" />
+    <parent
+      link="arm_left_link_3_e" />
+    <child
+      link="arm_left_link_4_u" />
+    <axis
+      xyz="0 0 -1" />
+    <limit effort="0" lower="-2.268928050994873" upper="2.268928050994873" velocity="1.1888351440429688"/>
+  </joint>
+  <link
+    name="arm_left_link_5_r">
+    <inertial>
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